File: pcb files/LED Weather Display.brd (EAGLE design)
At the start: 69.8 x 36.8 mm, 7 parts, among them IC1 74HCT245N, J1 POWER_JACK

Commit message: Update PCB files and documentation.
Parts:
- added PROGRAM: MOMENTARY-SWITCH-SPST-PTH-6.0MM, SparkFun-Switches:TACTILE_SWITCH_PTH_6.0MM
- added RESET: JST-XH-02-PIN-LONG-PAD, Rembrandt Electronics - JST XH Connectors v1-0:JST-XH-02-PACKAGE-LONG-PAD
- moved LEDS 12.0 mm to (49.5, 20.3)
- moved R1 11.5 mm to (40.6, 30.5)
- moved C1 11.4 mm to (63.5, 24.1)
- moved IC1 1.27 mm to (40.6, 15.2)
- moved SENSOR 1.27 mm to (49.5, 7.62)
Connections:
- new net N$7: PROGRAM.1, WEMOS1.RESET
- new net N$8: RESET.2, WEMOS1.D6
- net GND: now also PROGRAM.3, RESET.1
Routing:
- net N$8: track 0.00 -> 39.5 mm
- net N$7: track 0.00 -> 36.4 mm
- net N$1: track 63.5 -> 87.6 mm
- net GND: track 131.2 -> 142.8 mm
- net N$3: track 30.5 -> 21.6 mm
- net VCC: track 100.4 -> 93.0 mm
- net N$4: track 10.2 -> 16.5 mm
- net N$2: track 10.2 -> 15.2 mm
- net N$6: track 38.1 -> 34.3 mm
- net N$5: track 35.6 -> 31.8 mm

Commit message: PCB traces were incorrect for reset.
Connections:
- net N$7: now also WEMOS1.D6; no longer WEMOS1.RESET
- net N$8: now also WEMOS1.RESET; no longer WEMOS1.D6
Routing:
- net N$8: track 39.5 -> 29.4 mm
- net N$7: track 36.4 -> 46.0 mm
Changed lines of the file:
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@@
 <signal name="N$7">
 <contactref element="PROGRAM" pad="1"/>
-<contactref element="WEMOS1" pad="RESET"/>
-<wire x1="56.4388" y1="34.0106" x2="26.67" y2="34.0106" width="0.2032" layer="16"/>
-<wire x1="26.67" y1="34.0106" x2="26.67" y2="34.29" width="0.2032" layer="16"/>
-<wire x1="26.67" y1="34.29" x2="26.67" y2="27.94" width="0.2032" layer="16"/>
+<contactref element="WEMOS1" pad="D6"/>
+<wire x1="16.51" y1="34.0106" x2="16.51" y2="27.94" width="0.2032" layer="16"/>
+<wire x1="56.4388" y1="34.0106" x2="16.51" y2="34.0106" width="0.2032" layer="16"/>
 </signal>
 <signal name="N$8">
 <contactref element="RESET" pad="2"/>
-<contactref element="WEMOS1" pad="D6"/>
 <wire x1="49.53" y1="29.21" x2="49.53" y2="30.5308" width="0.2032" layer="1"/>
 <wire x1="49.53" y1="30.5308" x2="45.7962" y2="30.5308" width="0.2032" layer="1"/>
-<wire x1="45.7962" y1="30.5308" x2="45.7962" y2="31.8262" width="0.2032" layer="1"/>
-<wire x1="45.7962" y1="31.8262" x2="16.51" y2="31.8262" width="0.2032" layer="1"/>
-<wire x1="16.51" y1="31.8262" x2="16.51" y2="27.94" width="0.2032" layer="1"/>
+<wire x1="45.7962" y1="30.5308" x2="45.7962" y2="31.75" width="0.2032" layer="1"/>
+<contactref element="WEMOS1" pad="RESET"/>
+<wire x1="45.7962" y1="31.75" x2="45.7962" y2="31.8262" width="0.2032" layer="1"/>
+<wire x1="45.7962" y1="31.8262" x2="26.67" y2="31.8262" width="0.2032" layer="1"/>
+<wire x1="26.67" y1="31.8262" x2="26.67" y2="27.94" width="0.2032" layer="1"/>
 </signal>
 </signals>
